File: pcb/halogen32.kicad_pcb (KiCad board)
At the start: 2 copper layers, 8 parts, among them J1 Conn_ARM_JTAG_SWD_10, J2 USB_C_Receptacle_USB2.0_16P, J3 Conn_01x04_Socket, J4 Conn_01x16_Pin, J5 Conn_01x12_Pin, U1 STM32F411CEUx, U2 AMS1117-3.3

Commit message: Added DC jack and buck converter
Parts:
- removed D1: SK6805, LED_SMD:LED_SK6805_PLCC4_2.4x2.7mm_P1.3mm
- removed J1: Conn_ARM_JTAG_SWD_10, Connector_PinHeader_1.27mm:PinHeader_2x05_P1.27mm_Vertical
- removed J2: USB_C_Receptacle_USB2.0_16P, Connector_USB:USB_C_Receptacle_Amphenol_12401548E4-2A
- removed J3: Conn_01x04_Socket, Connector_JST:JST_SH_BM02B-SRSS-TB_1x02-1MP_P1.00mm_Vertical
- removed J4: Conn_01x16_Pin, Connector_PinSocket_2.54mm:PinSocket_1x16_P2.54mm_Vertical
- removed J5: Conn_01x12_Pin, Connector_PinSocket_2.54mm:PinSocket_1x12_P2.54mm_Vertical
- removed U1: STM32F411CEUx, Package_DFN_QFN:QFN-48-1EP_7x7mm_P0.5mm_EP5.6x5.6mm
- removed U2: AMS1117-3.3, Package_TO_SOT_SMD:SOT-223-3_TabPin2

Commit message: Assigned footprints and imported footprints into pcb layout.
Parts:
- added C1: 100n, Capacitor_SMD:CP_Elec_3x5.3, F.Cu at (18.6, 150.6)
- added C10: 10p, Capacitor_SMD:CP_Elec_3x5.3, F.Cu at (32.1, 155.4)
- added C11: 10p, Capacitor_SMD:CP_Elec_3x5.3, F.Cu at (32.1, 160.3)
- added C12: 1000u, Capacitor_SMD:CP_Elec_3x5.3, F.Cu at (32.1, 165.2)
- added C13: 22u, Capacitor_SMD:CP_Elec_3x5.3, F.Cu at (38.9, 150.6)
- added C14: 2.2u, Capacitor_SMD:CP_Elec_3x5.3, F.Cu at (38.9, 155.4)
- added C15: 2200u, Capacitor_SMD:CP_Elec_3x5.3, F.Cu at (38.9, 160.3)
- added C16: 100u, Capacitor_SMD:CP_Elec_3x5.3, F.Cu at (38.9, 165.2)
- added C2: 100n, Capacitor_SMD:CP_Elec_3x5.3, F.Cu at (18.6, 155.4)
- added C3: 100n, Capacitor_SMD:CP_Elec_3x5.3, F.Cu at (18.6, 160.3)
- added C4: 100n, Capacitor_SMD:CP_Elec_3x5.3, F.Cu at (18.6, 165.2)
- added C5: 10u, Capacitor_SMD:CP_Elec_3x5.3, F.Cu at (25.4, 150.6)
- added C6: 10n, Capacitor_SMD:CP_Elec_3x5.3, F.Cu at (25.4, 155.4)
- added C7: 1u, Capacitor_SMD:CP_Elec_3x5.3, F.Cu at (25.4, 160.3)
- added C8: 1u, Capacitor_SMD:CP_Elec_3x5.3, F.Cu at (25.4, 165.2)
- added C9: 22u, Capacitor_SMD:CP_Elec_3x5.3, F.Cu at (32.1, 150.6)
- added D1: SK6805, LED_SMD:LED_SK6805_PLCC4_2.4x2.7mm_P1.3mm, F.Cu at (58.1, 163.8)
- added D2: D, Diode_SMD:D_0201_0603Metric, F.Cu at (57.1, 166.7)
- added FB1: 120R, Ferrite_THT:LairdTech_28C0236-0JW-10, F.Cu at (54.6, 188.1)
- added H1: MountingHole, MountingHole:MountingHole_2.5mm, F.Cu at (18.5, 170.8)
- added H2: MountingHole, MountingHole:MountingHole_2.5mm, F.Cu at (18.5, 177.4)
- added H3: MountingHole, MountingHole:MountingHole_2.5mm, F.Cu at (18.5, 183.9)
- added H4: MountingHole, MountingHole:MountingHole_2.5mm, F.Cu at (18.5, 190.5)
- added J1: Conn_ARM_JTAG_SWD_10, Connector_PinHeader_1.27mm:PinHeader_2x05_P1.27mm_Vertical, F.Cu at (37.0, 181.6)
- added J2: USB_C_Receptacle_USB2.0_16P, Connector_USB:USB_C_Plug_Molex_105444, F.Cu at (50.6, 164.3)
- added J3: Conn_01x04_Pin, Connector_JST:JST_EH_B4B-EH-A_1x04_P2.50mm_Vertical, F.Cu at (49.3, 150.8)
- added J4: Conn_01x20_Socket, Connector_PinSocket_1.00mm:PinSocket_1x20_P1.00mm_Vertical, F.Cu at (23.8, 169.3)
- added J5: Conn_01x14_Socket, Connector_PinSocket_1.00mm:PinSocket_1x14_P1.00mm_Vertical, F.Cu at (44.3, 149.9)
- added J6: Barrel_Jack, Connector_BarrelJack:BarrelJack_CLIFF_FC681465S_SMT_Horizontal, F.Cu at (52.0, 175.6)
- added L1: 68u, Inductor_SMD:L_6.3x6.3_H3, F.Cu at (59.9, 157.9)
- added R1: 5.1k, Resistor_SMD:R_0201_0603Metric, F.Cu at (62.9, 184.5)
- added R2: 500, Resistor_SMD:R_0201_0603Metric, F.Cu at (62.9, 186.2)
- added R3: 5.1k, Resistor_SMD:R_0201_0603Metric, F.Cu at (62.9, 188.0)
- added R4: 5.1k, Resistor_SMD:R_0201_0603Metric, F.Cu at (62.9, 189.8)
- added R5: 5.1k, Resistor_SMD:R_0201_0603Metric, F.Cu at (62.9, 191.5)
- added SW1: SW_SPDT, Button_Switch_SMD:SW_SPST_TL3342, F.Cu at (30.1, 183.4)
- added SW2: SW_SPDT, Button_Switch_SMD:SW_SPST_TL3342, F.Cu at (30.1, 190.5)
- added U1: STM32F411CEUx, Package_DFN_QFN:QFN-48-1EP_7x7mm_P0.5mm_EP5.6x5.6mm, F.Cu at (48.1, 188.3)
- added U2: AMS1117-3.3, Package_TO_SOT_SMD:SOT-223-3_TabPin2, F.Cu at (50.7, 158.2)
- added U3: LM2576HVS-5, Package_TO_SOT_SMD:TO-263-5_TabPin3, F.Cu at (36.0, 173.8)
- added Y1: 16MHz, Crystal:Crystal_SMD_0603-2Pin_6.0x3.5mm, F.Cu at (38.9, 191.1)

Commit message: Began work on rough layout.
Parts:
- moved H1 151.2 mm to (151.0, 98.0)
- moved SW2 144.9 mm to (164.3, 135.9)
- moved SW1 140.0 mm to (164.3, 143.6)
- moved H3 137.8 mm to (150.5, 144.5)
- moved J6 131.8 mm to (163.0, 104.5)
- moved J2 125.4 mm to (169.6, 124.7), turned to 90 degrees
- moved D1 119.8 mm to (167.5, 115.2)
- moved H2 117.1 mm to (105.0, 98.5)
- moved U3 102.0 mm to (122.7, 119.9)
- moved U2 99.8 mm to (141.8, 117.5)
- moved H4 97.1 mm to (104.5, 145.5)
- moved FB1 96.7 mm to (136.4, 136.5)
- moved U1 95.4 mm to (124.2, 130.9)
- moved L1 86.6 mm to (140.8, 127.0)
- moved J1 79.9 mm to (105.3, 140.1), turned to 180 degrees
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